File: arduino/ArduinoProMini.NRF24.DHT/ArduinoProMini.NRF24.DHT.brd (EAGLE design)
At the start: 86 x 63.5 mm, 7 parts, among them U1 DHT22

Commit message: added schematic + board
Parts:
- moved U1 21.7 mm to (12.7, 10.2), turned to 0 degrees
- moved C1 17.7 mm to (40.6, 41.9)
- moved R1 11.4 mm to (25.4, 40.6), turned to 180 degrees
- moved U$2 4.58 mm to (26.7, 53.3)
- moved U$1 1.27 mm to (31.8, 26.7)
Connections:
- net N$2 renamed RAW
- net VCC renamed 3.3V
- net GND: now also U$1.GND, U$1.GND1
Routing:
- net 3.3V: track 50.5 -> 88.8 mm
- net GND: track 82.3 -> 118.0 mm
- net N$2: track 28.0 -> 43.9 mm
- net N$8: track 39.0 -> 49.1 mm, vias 0 -> 1
- net N$9: track 44.3 -> 48.1 mm
- net N$6: track 33.5 -> 36.6 mm
- net N$10: track 44.4 -> 47.2 mm
- net N$7: track 31.7 -> 34.1 mm
- net RAW: track 29.1 -> 29.7 mm
Other:
- board size 86 x 63.5 mm -> 88.6 x 63.5 mm
